File: RC6502 Apple 1 SBC/RC6502 Apple 1 SBC.sch (KiCad schematic (older format))
At the start: 48 parts, among them J1 VP GND, J10 RAM_EN, J11 PIA_EN, J2 Arduino Nano, J3 Backplane, J4 Hole, J5 Hole, J6 Hole, J7 Hole, J8 Power, J9 ROM_EN, SW1 RESET, U1 6502, U2 HM62256BLP-7, U3 74HCT138, U4 28C256, U5 74HCT00, U6 NE555, U7 74HCT04, U8 6821, U9 MCP23S17, X1 1MHz

Commit message: Fixed dowload types hex asm bas
Parts:
- A13, A14, J10, J11, J9: symbol Jumper_NC_Dual -> RC6502-Apple-1-SBC-rescue:Jumper_NC_Dual
- C1, C11, C12, C2, C3, C4, C5, C6, C7, C8, C9: symbol C -> RC6502-Apple-1-SBC-rescue:C
- C10: symbol CP -> RC6502-Apple-1-SBC-rescue:CP
- D1: symbol LED -> RC6502-Apple-1-SBC-rescue:LED
- J1, J8: symbol CONN_01X02 -> RC6502-Apple-1-SBC-rescue:CONN_01X02
- J2: symbol Arduino_Nano_Header -> RC6502-Apple-1-SBC-rescue:Arduino_Nano_Header
- J3: symbol RC6502_Backplane -> RC6502-Apple-1-SBC-rescue:RC6502_Backplane
- J4, J5, J6, J7: symbol CONN_01X01 -> RC6502-Apple-1-SBC-rescue:CONN_01X01
- JP1: symbol Jumper_NC_Small -> RC6502-Apple-1-SBC-rescue:Jumper_NC_Small
- R1, R10, R2, R3, R4, R5, R6, R7, R8, R9: symbol R -> RC6502-Apple-1-SBC-rescue:R
- SW1: symbol SW_SPST -> RC6502-Apple-1-SBC-rescue:SW_SPST
- U1: symbol 6502 -> RC6502-Apple-1-SBC-rescue:6502
- U2: symbol HM62256BLP-7 -> RC6502-Apple-1-SBC-rescue:HM62256BLP-7
- U3: symbol 74LS138 -> RC6502-Apple-1-SBC-rescue:74LS138
- U4: symbol 28C256 -> RC6502-Apple-1-SBC-rescue:28C256
- U5: symbol 74HCT00 -> RC6502-Apple-1-SBC-rescue:74HCT00
- U6: symbol NE555 -> RC6502-Apple-1-SBC-rescue:NE555
- U7: symbol 74LS04 -> RC6502-Apple-1-SBC-rescue:74LS04
- U8: symbol MC6821 -> RC6502-Apple-1-SBC-rescue:MC6821
- U9: symbol MCP23S17 -> RC6502-Apple-1-SBC-rescue:MCP23S17
- X1: symbol ACO-xxxMHz -> RC6502-Apple-1-SBC-rescue:ACO-xxxMHz
Connections:
- wire segments 158 -> 207
