File: RC6502 PSG/RC6502 PSG.sch (KiCad schematic (older format))
At the start: 28 parts, among them J1 TRS_3.5mm, J2 Port, J3 Base, J4 RC6502_Backplane, J5 EXT, U1 LM386, U2 74LS244, U3 74LS138, U4 74LS138, U5 SN76489AN, U6 74LS374, U7 74LS374, X1 TCXO-14

Commit message: Update Kicad libs
Parts:
- C1, C3, C8: symbol CP -> Device:CP
- C10, C11, C12, C13, C14, C4, C7, C9: symbol C -> Device:C
- J1: symbol TRS_3.5mm -> RC6502-PSG-rescue:TRS_3.5mm
- J2, J3: symbol Conn_02x08_Odd_Even -> RC6502-PSG-rescue:Conn_02x08_Odd_Even
- J4: symbol RC6502_Backplane -> RC6502-PSG-rescue:RC6502_Backplane
- J5: symbol Conn_01x02 -> RC6502-PSG-rescue:Conn_01x02
- JP1, JP2: symbol Jumper_NO_Small -> Device:Jumper_NO_Small
- LS1: symbol Speaker -> Device:Speaker
- R2: symbol R -> Device:R
- U1: symbol LM386 -> RC6502-PSG-rescue:LM386
- U2: symbol 74LS244 -> RC6502-PSG-rescue:74LS244
- U3, U4: symbol 74LS138 -> RC6502-PSG-rescue:74LS138
- U5: symbol SN76489AN -> SN76489AN:SN76489AN
- U6, U7: symbol 74LS374 -> RC6502-PSG-rescue:74LS374
- X1: symbol TCXO-14 -> RC6502-PSG-rescue:TCXO-14
Connections:
- wire segments 185 -> 220
